File: DFB1/kicad5/dfb1_r5/dfb1_r5.kicad_pcb (KiCad board)
At the start: 4 copper layers, 169 x 71.4 mm, 79 parts, among them IC1 IS42S16320D-7TL, IC2 IS42S16320D-7TL, IC3 SN74CB3T3245PW, IC4 SN74CB3T3245PW, IC5 SN74CB3T3245PW, IC6 SN74CB3T3245PW, J1 Conn_01x50, J2 Conn_02x04_Odd_Even, J3 Conn_01x30, J4 Conn_02x03_Odd_Even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

Commit message: Original PCB design file with silkscreen touchup
Original PCB design file with silkscreen touchup
Connections:
- net /~EXPD renamed /~{EXPD}
- net /~IACK renamed /~{IACK}
- net /~MFP_IEI renamed /~{MFP_IEI}
- net /~MFP_INT renamed /~{MFP_INT}
- net /~XINT1 renamed /~{XINT1}
- net /~XINT3 renamed /~{XINT3}
- net XR~W renamed XR~{W}
- net ~AS renamed ~{AS}
- net ~AVEC renamed ~{AVEC}
- net ~BERR renamed ~{BERR}
- net ~BG renamed ~{BG}
- net ~BGK renamed ~{BGK}
- net ~BOE renamed ~{BOE}
- net ~BR renamed ~{BR}
- net ~CAS renamed ~{CAS}
- net ~CBACK renamed ~{CBACK}
- net ~CBREQ renamed ~{CBREQ}
- net ~DS renamed ~{DS}
- net ~DSACK0 renamed ~{DSACK0}
- net ~DSACK1 renamed ~{DSACK1}
- net ~FPUCS renamed ~{FPUCS}
- net ~FPUDSACK0 renamed ~{FPUDSACK0}
- net ~FPUDSACK1 renamed ~{FPUDSACK1}
- net ~HLT renamed ~{HLT}
- net ~IPL0 renamed ~{IPL0}
- net ~IPL1 renamed ~{IPL1}
- net ~IPL2 renamed ~{IPL2}
- net ~LDS renamed ~{LDS}
- net ~RAMWE renamed ~{RAMWE}
- net ~RAS renamed ~{RAS}
- net ~ROMCE renamed ~{ROMCE}
- net ~ROMOE renamed ~{ROMOE}
- net ~RST renamed ~{RST}
- net ~STERM renamed ~{STERM}
- net ~UDS renamed ~{UDS}
- net ~XAS renamed ~{XAS}
- net ~XBG renamed ~{XBG}
- net ~XBGK renamed ~{XBGK}
- net ~XBR renamed ~{XBR}
- net ~XDTACK renamed ~{XDTACK}
- net ~XHALT renamed ~{XHALT}
Other:
- net class CLK removed
- net class Default removed
- net class PWR removed
- board text added: "2025-08-01 Assembled by Suavek"
- board text added: "DFB1"
- board text removed: "~DFB1"
